File: Hardware/soilsync/untitled.kicad_sch (KiCad schematic)
At the start: 0 parts

Commit message: layout nearly finished.
need to add mosfet and programming connector
Parts:
- added J10, J11, J2, J3, J4, J5, J6, J7, J8, J9: Screw_Terminal_01x03, TerminalBlock_4Ucon:TerminalBlock_4Ucon_1x03_P3.50mm_Horizontal, symbol Connector:Screw_Terminal_01x03
- added R1, R11, R13, R15, R17, R19, R3, R5, R7, R9: 4.7k, Resistor_SMD:R_0805_2012Metric, symbol Device:R
- added R10, R12, R14, R16, R18, R2, R20, R4, R6, R8: 8.2k, Resistor_SMD:R_0805_2012Metric, symbol Device:R
Connections:
- new net: J7.3 (Pin_3), R11.1, R12.1
- new net: J2.3 (Pin_3), R1.1, R2.1
- new net: J11.3 (Pin_3), R19.1, R20.1
- new net: J5.3 (Pin_3), R7.1, R8.1
- new net: J4.3 (Pin_3), R5.1, R6.1
- new net: J3.3 (Pin_3), R3.1, R4.1
- new net: J10.3 (Pin_3), R17.1, R18.1
- new net: J9.3 (Pin_3), R15.1, R16.1
- new net: J8.3 (Pin_3), R13.1, R14.1
- new net: J6.3 (Pin_3), R10.1, R9.1
- new net +5V: J10.2 (Pin_2), J11.2 (Pin_2), J2.2 (Pin_2), J3.2 (Pin_2), J4.2 (Pin_2), J5.2 (Pin_2), J6.2 (Pin_2), J7.2 (Pin_2), J8.2 (Pin_2), J9.2 (Pin_2)
- new net GND: J10.1 (Pin_1), J11.1 (Pin_1), J2.1 (Pin_1), J3.1 (Pin_1), J4.1 (Pin_1), J5.1 (Pin_1), J6.1 (Pin_1), J7.1 (Pin_1), J8.1 (Pin_1), J9.1 (Pin_1), R10.2, R12.2, R14.2, R16.2, R18.2, R2.2, R20.2, R4.2, R6.2, R8.2
- new net SENSOR_1: R1.2
- new net SENSOR_10: R19.2
- new net SENSOR_2: R3.2
- new net SENSOR_3: R5.2
- new net SENSOR_4: R7.2
- new net SENSOR_5: R9.2
- new net SENSOR_6: R11.2
- new net SENSOR_7: R13.2
- new net SENSOR_8: R15.2
- new net SENSOR_9: R17.2
